Commit message: ur_gripper urdf add

File: Universal_Robots_ROS_Driver/ur_description/urdf/ur.ros2_control.xacro (robot description, xacro)
@@ -122,4 +122,11 @@
         <state_interface name="effort"/>
         <param name="initial_position">${initial_positions['wrist_3_joint']}</param>  <!-- initial position for the FakeSystem -->
+      </joint>
+      <joint name="robotiq_85_left_knuckle_joint">
+        <command_interface name="position"/>
+        <state_interface name="position">
+          <param name="initial_value">${initial_positions['robotiq_85_left_knuckle_joint']}</param>
+        </state_interface>
+        <state_interface name="velocity"/>
       </joint>
       <sensor name="tcp_fts_sensor">
